File: core_board/core_board.kicad_sch (KiCad schematic)
At the start: 36 parts, among them J1 Conn_01x13_Socket, J2 Conn_01x13_Socket, J3 Ignitor Output, J4 Micro_SD_Card, J5 Battery Input, J7 Connector 1, J8 Connector 2, U1 CPC1002N, U2 CPC1002N, U3 CPC1002N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

Commit message: Fixed connector compatibility with STEMMA QT and Qwiic
Parts:
- J7, J8: footprint Connector_Molex:Molex_PicoBlade_53047-0410_1x04_P1.25mm_Vertical -> G2Custom:JST_SH_BM04B-SRSS-TB_1x04-1MP_P1.00mm_Vertical-CUSTOM
Connections:
- net +3.3V: now also J7.3 (Pin_3), J8.3 (Pin_3); no longer J7.1 (Pin_1), J8.1 (Pin_1)
- net SCL Inter Board: now also J7.1 (Pin_1), J8.1 (Pin_1); no longer J7.2 (Pin_2), J8.2 (Pin_2)
- net SDA Inter Board: now also J7.2 (Pin_2), J8.2 (Pin_2); no longer J7.3 (Pin_3), J8.3 (Pin_3)

Commit message: Corrected DRC errors
Parts:
- Y1: value 33.768kHz -> 32.768kHz
Changed lines of the file:
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@@
 			)
 		)
-		(property "Value" "33.768kHz"
+		(property "Value" "32.768kHz"
 			(at 266.446 106.934 0)
 			(effects

Commit message: Added Aerospace Club logo and gave mounting holes pads
Parts:
- H1, H2, H3: footprint MountingHole:MountingHole_2.2mm_M2_ISO7380 -> MountingHole:MountingHole_2.2mm_M2_ISO7380_Pad
Changed lines of the file:
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@@
 			)
 		)
-		(property "Footprint" "MountingHole:MountingHole_2.2mm_M2_ISO7380"
+		(property "Footprint" "MountingHole:MountingHole_2.2mm_M2_ISO7380_Pad"
 			(at 16.51 175.26 0)
 			(effects
@@
 			)
 		)
-		(property "Footprint" "MountingHole:MountingHole_2.2mm_M2_ISO7380"
+		(property "Footprint" "MountingHole:MountingHole_2.2mm_M2_ISO7380_Pad"
 			(at 16.51 168.91 0)
 			(effects
@@
 			)
 		)
-		(property "Footprint" "MountingHole:MountingHole_2.2mm_M2_ISO7380"
+		(property "Footprint" "MountingHole:MountingHole_2.2mm_M2_ISO7380_Pad"
 			(at 16.51 181.61 0)
 			(effects

Commit message: Tweaked mounting holes, removed warning on back
Parts:
- added H4: MountingHole, MountingHole:MountingHole_2.2mm_M2_ISO7380_Pad, symbol Mechanical:MountingHole
Changed lines of the file:
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@@
+	)
+	(symbol
+		(lib_id "Mechanical:MountingHole")
+		(at 16.51 187.96 0)
+		(unit 1)
+		(exclude_from_sim yes)
+		(in_bom no)
+		(on_board yes)
+		(dnp no)
+		(fields_autoplaced yes)
+		(property "Reference" "H4"
+			(at 19.05 186.6899 0)
+			(effects
+				(font
+					(size 1.27 1.27)
+				)
+				(justify left)
+			)
+		)
+		(property "Value" "MountingHole"
+			(at 19.05 189.2299 0)
+			(effects
+				(font
+					(size 1.27 1.27)
+				)
+				(justify left)
+			)
+		)
+		(property "Footprint" "MountingHole:MountingHole_2.2mm_M2_ISO7380_Pad"
+			(at 16.51 187.96 0)
+			(effects
+				(font
+					(size 1.27 1.27)
+				)
+				(hide yes)
+			)
+		)
+		(property "Datasheet" "~"
+			(at 16.51 187.96 0)
+			(effects
+				(font
+					(size 1.27 1.27)
+				)
+				(hide yes)
+			)
+		)
+		(property "Description" "Mounting Hole without connection"
+			(at 16.51 187.96 0)
+			(effects
+				(font
+					(size 1.27 1.27)
+				)
+				(hide yes)
+			)
+		)
+		(instances
+			(project "core_board"
+				(path "/d1f95e7e-c47f-4536-a77e-9f553fe58a7a"
+					(reference "H4")
+					(unit 1)
+				)
+			)
+		)
 	)
 	(symbol
